Commit message: migrated the robot to be used in the gazebo ignition simulation and added functionalities for a lidar

File: mtt_ws/src/mtt_description/urdf/robot.urdf.xacro (robot description, xacro)
@@ -1331,8 +1331,77 @@
         <material>Gazebo/Orange</material>
     </gazebo>
-    <gazebo>
-        <plugin filename="libgazebo_ros2_control.so" name="gazebo_ros2_control">
-            <parameters>$(find the_mtt_bringup)/config/control.yaml</parameters>
-        </plugin>
-    </gazebo>
+<!-- LiDAR Link -->
+<link name="lidar_link">
+  <pose>0 0 0.2 0 0 0</pose>
+  <visual>
+    <geometry>
+      <cylinder length="0.05" radius="0.02"/>
+    </geometry>
+    <material name="green">
+      <color rgba="0 1 0 1"/>
+    </material>
+  </visual>
+  <collision>
+    <geometry>
+      <cylinder length="0.05" radius="0.02"/>
+    </geometry>
+  </collision>
+  <inertial>
+    <mass value="0.1"/>
+    <inertia ixx="0.0001" ixy="0.0" ixz="0.0"
+             iyy="0.0001" iyz="0.0"
+             izz="0.0001"/>
+  </inertial>
+</link>
+<!-- Joint to attach LiDAR to base_footprint -->
+<joint name="lidar_joint" type="fixed">
+  <parent link="base_footprint"/>
+  <child link="lidar_link"/>
+  <origin xyz="0 0 0.8" rpy="0 0 0"/>
+</joint>
+<!-- Gazebo sensor plugin -->
+<gazebo reference="lidar_link">
+  <sensor name="lidar" type="gpu_lidar">
+    <pose>0 0 0 0 0 0</pose>
+    <update_rate>10</update_rate>
+    <ray>
+      <scan>
+        <horizontal>
+          <samples>360</samples>
+          <resolution>1.0</resolution>
+          <min_angle>-3.14</min_angle>
+          <max_angle>3.14</max_angle>
+        </horizontal>
+      </scan>
+      <range>
+        <min>0.1</min>
+        <max>30.0</max>
+      </range>
+    </ray>
+    <plugin name="gz_ros_lidar" filename="gz-ros2-laser-scan-system">
+        <ros_topic>/scan</ros_topic>
+        <ros_type>sensor_msgs/msg/LaserScan</ros_type>
+        <gz_type>gz.msgs.LaserScan</gz_type>
+        <frame_name>lidar_link</frame_name>
+    </plugin>
+  </sensor>
+</gazebo>
+<gazebo>
+  <plugin name="p3d_base_odom" filename="libgazebo_ros_p3d.so">
+    <ros>
+      <remapping>odom:=/odom</remapping>
+    </ros>
+    <robotNamespace>/</robotNamespace>
+    <bodyName>base_link</bodyName>   <!-- Or base_footprint, if that’s your main body -->
+    <frameName>odom</frameName>
+    <updateRate>50.0</updateRate>
+    <gaussianNoise>0.01</gaussianNoise>
+    <alwaysOn>true</alwaysOn>
+  </plugin>
+  <plugin
+    filename="gz-sim-pose-publisher-system"
+    name="gz::sim::systems::PosePublisher">
+  <publish_model_pose>true</publish_model_pose>
+</plugin>
+</gazebo>
 </robot>

Commit message: log warn level

File: mtt_ws/src/mtt_description/urdf/robot.urdf.xacro (robot description, xacro)
@@ -1,4 +1,4 @@
 <?xml version="1.0"?>
-<robot name="onshape"  xmlns:xacro="https://www.ros.org/wiki/xacro">
+<robot name="mtt_robot"  xmlns:xacro="https://www.ros.org/wiki/xacro">
     <xacro:macro name="default_transmission" params="joint_name">
         <transmission name="transmission_${joint_name}">
@@ -10,5 +10,12 @@
         </transmission>
     </xacro:macro>
-    <link name="base_footprint"/>
+        <link name="base_footprint"/>
+        <!-- Add a base_link alias (Nav2 expects base_link). base_link coincides with base_footprint origin. -->
+        <link name="base_link"/>
+        <joint name="base_link_joint" type="fixed">
+            <parent link="base_footprint"/>
+            <child link="base_link"/>
+            <origin xyz="0 0 0" rpy="0 0 0"/>
+        </joint>
     <link name="MTT_body">
     <visual>
@@ -1393,3 +1400,16 @@
 </plugin>
 </gazebo>
+<!-- Ground-truth odometry publisher -->
+<gazebo>
+        <plugin filename="gz-sim-odometry-publisher-system" name="gz::sim::systems::OdometryPublisher">
+            <odom_frame>odom</odom_frame>
+            <!-- Publish odom->base_link -->
+            <robot_base_frame>base_link</robot_base_frame>
+        <odom_publish_frequency>50</odom_publish_frequency>
+        <dimensions>3</dimensions>
+        <xyz_offset>0 0 0</xyz_offset>
+        <rpy_offset>0 0 0</rpy_offset>
+        <gaussian_noise>0</gaussian_noise>
+    </plugin>
+</gazebo>
 </robot>

Commit message: changed the link name mtt_body to base_link

File: mtt_ws/src/mtt_description/urdf/robot.urdf.xacro (robot description, xacro)
@@ -11,5 +11,5 @@
     </xacro:macro>
     <link name="base_footprint"/>
-    <link name="MTT_body">
+    <link name="base_link">
     <visual>
     <origin xyz="-0.0034808381178577409154 -0.051022168970358453 0.49330103716210749187" rpy="0 -0 3.1415926535897926719" />
@@ -34,6 +34,6 @@
     </link>
    <joint name="base_joint" type="fixed">
-    <parent link="base_footprint"/>
-    <child link="MTT_body"/>
+    <parent link="base_link"/>
+    <child link="base_footprint"/>
     <origin xyz="0 0 0.1" rpy="0 0 0"/>
     </joint>
@@ -62,5 +62,5 @@
     <joint name="1_continuous" type="continuous">
     <origin xyz="0.7014675763219452298 -0.30260966897135904707 0.29942602155526376606" rpy="1.570796326794896558 -0 -7.5633943552588769595e-16" />
-    <parent link="MTT_body" />
+    <parent link="base_link" />
     <child link="Rouleau_track_1" />
     <axis xyz="0 0 1"/>
@@ -100,5 +100,5 @@
     <joint name="2_continuous" type="continuous">
     <origin xyz="0.63021293776953013488 -0.30260966897135899156 0.24925922731169392055" rpy="1.570796326794896558 -0 -7.5633943552588769595e-16" />
-    <parent link="MTT_body" />
+    <parent link="base_link" />
     <child link="Rouleau_track_2" />
     <axis xyz="0 0 1"/>
@@ -138,5 +138,5 @@
     <joint name="3_continuous" type="continuous">
     <origin xyz="0.55767703136521962204 -0.30260966897135893605 0.20171053820694723191" rpy="1.570796326794896558 -0 -7.5633943552588769595e-16" />
-    <parent link="MTT_body" />
+    <parent link="base_link" />
     <child link="Rouleau_track_3" />
     <axis xyz="0 0 1"/>
@@ -176,5 +176,5 @@
     <joint name="4_continuous" type="continuous">
     <origin xyz="0.47434412390430480411 -0.30260966897135888054 0.17622412429685807567" rpy="1.570796326794896558 -0 -7.5633943552588769595e-16" />
-    <parent link="MTT_body" />
+    <parent link="base_link" />
     <child link="Rouleau_track_4" />
     <axis xyz="0 0 1"/>
@@ -214,5 +214,5 @@
     <joint name="5_continuous" type="continuous">
     <origin xyz="0.39101121644338021621 -0.30260966897135876952 0.15073771038676886391" rpy="1.570796326794896558 -0 -7.5633943552588769595e-16" />
-    <parent link="MTT_body" />
+    <parent link="base_link" />
     <child link="Rouleau_track_5" />
     <axis xyz="0 0 1"/>
@@ -252,5 +252,5 @@
     <joint name="6_continuous" type="continuous">
     <origin xyz="0.30589785624702453548 -0.30260966897135871401 0.13716525069048957075" rpy="1.570796326794896558 -0 -7.5633943552588769595e-16" />
-    <parent link="MTT_body" />
+    <parent link="base_link" />
     <child link="Rouleau_track_6" />
     <axis xyz="0 0 1"/>
@@ -290,5 +290,5 @@
     <joint name="7_continuous" type="continuous">
     <origin xyz="0.21875469438405417688 -0.3026096689713586585 0.13717527124629197433" rpy="1.570796326794896558 -0 -7.5633943552588769595e-16" />
-    <parent link="MTT_body" />
+    <parent link="base_link" />
     <child link="Rouleau_track_7" />
     <axis xyz="0 0 1"/>
@@ -328,5 +328,5 @@
     <joint name="8_continuous" type="continuous">
     <origin xyz="0.13161153252108562239 -0.3026096689713586585 0.13718529180209448892" rpy="1.570796326794896558 -0 -7.5633943552588769595e-16" />
-    <parent link="MTT_body" />
+    <parent link="base_link" />
     <child link="Rouleau_track_8" />
     <axis xyz="0 0 1"/>
@@ -366,5 +366,5 @@
     <joint name="9_continuous" type="continuous">
     <origin xyz="0.044468370658119274474 -0.30260966897135854747 0.13719531235789694801" rpy="1.570796326794896558 -0 -7.5633943552588769595e-16" />
-    <parent link="MTT_body" />
+    <parent link="base_link" />
     <child link="Rouleau_track_9" />
     <axis xyz="0 0 1"/>
@@ -404,5 +404,5 @@
     <joint name="10_continuous" type="continuous">
     <origin xyz="-0.042674791204848093462 -0.30260966897135843645 0.13720533291369940709" rpy="1.570796326794896558 -0 -7.5633943552588769595e-16" />
-    <parent link="MTT_body" />
+    <parent link="base_link" />
     <child link="Rouleau_track_10" />
     <axis xyz="0 0 1"/>
@@ -442,5 +442,5 @@
     <joint name="11_continuous" type="continuous">
     <origin xyz="-0.12981795306781560018 -0.30260966897135843645 0.13721535346950286538" rpy="1.570796326794896558 -0 -7.5633943552588769595e-16" />
-    <parent link="MTT_body" />
+    <parent link="base_link" />
     <child link="Rouleau_track_11" />
     <axis xyz="0 0 1"/>
@@ -480,5 +480,5 @@
     <joint name="12_continuous" type="continuous">
     <origin xyz="-0.21696111493078301669 -0.30260966897135832543 0.13722537402530532447" rpy="1.570796326794896558 -0 -7.5633943552588769595e-16" />
-    <parent link="MTT_body" />
+    <parent link="base_link" />
     <child link="Rouleau_track_12" />
     <axis xyz="0 0 1"/>
@@ -518,5 +518,5 @@
     <joint name="13_continuous" type="continuous">
     <origin xyz="-0.30410427679375034993 -0.30260966897135821441 0.13723539458110778355" rpy="1.570796326794896558 -0 -7.5633943552588769595e-16" />
-    <parent link="MTT_body" />
+    <parent link="base_link" />
     <child link="Rouleau_track_13" />
     <axis xyz="0 0 1"/>
@@ -556,5 +556,5 @@
     <joint name="14_continuous" type="continuous">
     <origin xyz="-0.39124743865671768317 -0.30260966897135821441 0.13724541513691029815" rpy="1.570796326794896558 -0 -7.5633943552588769595e-16" />
-    <parent link="MTT_body" />
+    <parent link="base_link" />
     <child link="Rouleau_track_14" />
     <axis xyz="0 0 1"/>
@@ -594,5 +594,5 @@
     <joint name="15_continuous" type="continuous">
     <origin xyz="-0.47839060051968412823 -0.30260966897135821441 0.13725543569271270172" rpy="1.570796326794896558 -0 -7.5633943552588769595e-16" />
-    <parent link="MTT_body" />
+    <parent link="base_link" />
     <child link="Rouleau_track_15" />
     <axis xyz="0 0 1"/>
@@ -632,5 +632,5 @@
     <joint name="16_continuous" type="continuous">
     <origin xyz="-0.56553376238265151699 -0.30260966897135799236 0.13726545624851521632" rpy="1.570796326794896558 -0 -7.5633943552588769595e-16" />
-    <parent link="MTT_body" />
+    <parent link="base_link" />
     <child link="Rouleau_track_16" />
     <axis xyz="0 0 1"/>
@@ -670,5 +670,5 @@
     <joint name="17_continuous" type="continuous">
     <origin xyz="-0.65267692424561885023 -0.30260966897135799236 0.13727547680431761989" rpy="1.570796326794896558 -0 -7.5633943552588769595e-16" />
-    <parent link="MTT_body" />
+    <parent link="base_link" />
     <child link="Rouleau_track_17" />
     <axis xyz="0 0 1"/>
@@ -708,5 +708,5 @@
     <joint name="18_continuous" type="continuous">
     <origin xyz="-0.73982008610858640552 -0.30260966897135788134 0.13728549736012013449" rpy="1.570796326794896558 -0 -7.5633943552588769595e-16" />
-    <parent link="MTT_body" />
+    <parent link="base_link" />
     <child link="Rouleau_track_18" />
     <axis xyz="0 0 1"/>
@@ -746,5 +746,5 @@
     <joint name="19_continuous" type="continuous">
     <origin xyz="-0.82595460894701899779 -0.30260966897135777032 0.14666682073043030288" rpy="1.570796326794896558 -0 -7.5633943552588769595e-16" />
-    <parent link="MTT_body" />
+    <parent link="base_link" />
     <child link="Rouleau_track_19" />
     <axis xyz="0 0 1"/>
@@ -784,5 +784,5 @@
     <joint name="20_continuous" type="continuous">
     <origin xyz="-0.91110403062049183376 -0.30260966897135777032 0.16520075578373016878" rpy="1.570796326794896558 -0 -7.5633943552588769595e-16" />
-    <parent link="MTT_body" />
+    <parent link="base_link" />
     <child link="Rouleau_track_20" />
     <axis xyz="0 0 1"/>
@@ -1117,5 +1117,5 @@
     <joint name="pitch" type="revolute">
     <origin xyz="-1.0511878376018575221 0.21250283103064232515 0.35775105114691785335" rpy="-1.570796326794896558 -0 -7.5633943552588769595e-16" />
-    <parent link="MTT_body" />
+    <parent link="base_link" />
     <child link="Frame_fixation_articule" />
     <axis xyz="0 0 1"/>
@@ -1319,5 +1319,5 @@
     <xacro:default_transmission joint_name="20_continuous"/>
     <xacro:default_transmission joint_name="yaw"/>
-    <gazebo reference="MTT_body">
+    <gazebo reference="base_link">
         <material>Gazebo/Orange</material>
     </gazebo>
@@ -1356,5 +1356,5 @@
 <!-- Joint to attach LiDAR to base_footprint -->
 <joint name="lidar_joint" type="fixed">
-  <parent link="base_footprint"/>
+  <parent link="base_link"/>
   <child link="lidar_link"/>
   <origin xyz="0 0 0.8" rpy="0 0 0"/>

Commit message: feat: MTT driver teleop/joint prototype - TF & odometry mockup working

File: mtt_ws/src/mtt_description/urdf/robot.urdf.xacro (robot description, xacro)
@@ -34,7 +34,7 @@
     </link>
    <joint name="base_joint" type="fixed">
-    <parent link="base_link"/>
-    <child link="base_footprint"/>
-    <origin xyz="0 0 0.1" rpy="0 0 0"/>
+    <parent link="base_footprint"/>
+    <child link="base_link"/>
+    <origin xyz="0 0 -0.1" rpy="0 0 0"/>
     </joint>
     <link name="Rouleau_track_1">

Commit message: urdf : add a ref point on robot

File: mtt_ws/src/mtt_description/urdf/robot.urdf.xacro (robot description, xacro)
@@ -13,5 +13,5 @@
     <link name="base_link">
     <visual>
-    <origin xyz="-0.0034808381178577409154 -0.051022168970358453 0.49330103716210749187" rpy="0 -0 3.1415926535897926719" />
+    <origin xyz="-0.0034808381178577409154 -0.051022168970358453 0.49330103716210749187" rpy="0 -0 ${pi}" />
     <geometry>
     <mesh filename="file://$(find mtt_description)/meshes/visual/m500_ra-02_r02.stl"/>
@@ -22,5 +22,5 @@
     </visual>
     <collision>
-    <origin xyz="-0.0034808381178577409154 -0.051022168970358453 0.49330103716210749187" rpy="0 -0 3.1415926535897926719" />
+    <origin xyz="-0.0034808381178577409154 -0.051022168970358453 0.49330103716210749187" rpy="0 -0 ${pi}" />
     <geometry>
     <mesh filename="file://$(find mtt_description)/meshes/collision/boitecollisionmtt_simple.stl"/>
@@ -1354,5 +1354,94 @@
   </inertial>
 </link>
-<!-- Joint to attach LiDAR to base_footprint -->
+<!-- Physical pencil mark reference point -->
+<link name="reference_point">
+  <visual>
+    <origin xyz="0 0 0" rpy="0 0 0"/>
+    <geometry>
+      <sphere radius="0.005"/>
+    </geometry>
+    <material name="mark_material">
+      <color rgba="1.0 0.0 0.0 1.0"/>
+    </material>
+  </visual>
+</link>
+<joint name="reference_point_joint" type="fixed">
+  <parent link="base_link"/>
+  <child link="reference_point"/>
+  <origin xyz="-0.7174808381178577409 0.21597831029643155 0.52330103716210749187" rpy="0 0 0"/>
+</joint>
+<!-- Center LiDAR -->
+<link name="center_lidar_link">
+  <visual>
+    <origin xyz="0 0 0" rpy="0 0 0"/>
+    <geometry>
+      <cylinder radius="0.05" length="0.1"/>
+    </geometry>
+    <material name="lidar_material">
+      <color rgba="0.2 0.2 0.2 1.0"/>
+    </material>
+  </visual>
+  <inertial>
+    <origin xyz="0 0 0" rpy="0 0 0"/>
+    <mass value="0.1"/>
+    <inertia ixx="0.0001" ixy="0.0" ixz="0.0"
+             iyy="0.0001" iyz="0.0"
+             izz="0.0001"/>
+  </inertial>
+</link>
+<joint name="center_lidar_joint" type="fixed">
+  <parent link="reference_point"/>
+  <child link="center_lidar_link"/>
+  <origin xyz="0.62 -0.266 0.355" rpy="0 0 ${pi/2}"/>
+</joint>
+<!-- Front LiDAR -->
+<link name="front_lidar_link">
+  <visual>
+    <origin xyz="0 0 0" rpy="0 0 0"/>
+    <geometry>
+      <cylinder radius="0.05" length="0.1"/>
+    </geometry>
+    <material name="lidar_material">
+      <color rgba="0.2 0.2 0.2 1.0"/>
+    </material>
+  </visual>
+  <inertial>
+    <origin xyz="0 0 0" rpy="0 0 0"/>
+    <mass value="0.1"/>
+    <inertia ixx="0.0001" ixy="0.0" ixz="0.0"
+             iyy="0.0001" iyz="0.0"
+             izz="0.0001"/>
+  </inertial>
+</link>
+<joint name="front_lidar_joint" type="fixed">
+  <parent link="reference_point"/>
+  <child link="front_lidar_link"/>
+  <origin xyz="1.24 -0.266 0.3302" rpy="0 0 0"/>
+</joint>
+<!-- Rear LiDAR -->
+<link name="rear_lidar_link">
+  <visual>
+    <origin xyz="0 0 0" rpy="0 0 0"/>
+    <geometry>
+      <cylinder radius="0.05" length="0.1"/>
+    </geometry>
+    <material name="lidar_material">
+      <color rgba="0.2 0.2 0.2 1.0"/>
+    </material>
+  </visual>
+  <inertial>
+    <origin xyz="0 0 0" rpy="0 0 0"/>
+    <mass value="0.1"/>
+    <inertia ixx="0.0001" ixy="0.0" ixz="0.0"
+             iyy="0.0001" iyz="0.0"
+             izz="0.0001"/>
+  </inertial>
+</link>
+<joint name="rear_lidar_joint" type="fixed">
+  <parent link="reference_point"/>
+  <child link="rear_lidar_link"/>
+  <origin xyz="0.01 -0.266 0.3302" rpy="0 0 0"/>
+</joint>
+<!-- Legacy LiDAR (kept for compatibility) -->
 <joint name="lidar_joint" type="fixed">
   <parent link="base_link"/>
@@ -1365,7 +1454,49 @@
 </plugin>
 </gazebo>
-<!-- Gazebo sensor plugin -->
-<gazebo reference="lidar_link">
-  <sensor name="lidar" type="gpu_lidar">
+<!-- Gazebo sensor plugin for Center LiDAR -->
+<gazebo reference="center_lidar_link">
+  <sensor name="center_lidar" type="gpu_lidar">
+    <pose>0 0 0 0 0 0</pose>
+    <update_rate>10</update_rate>
+    <ray>
+      <scan>
+        <horizontal>
+          <samples>360</samples>
+          <resolution>1.0</resolution>
+          <min_angle>-3.14</min_angle>
+          <max_angle>3.14</max_angle>
+        </horizontal>
+      </scan>
+      <range>
+        <min>0.1</min>
+        <max>30.0</max>
+      </range>
+    </ray>
+  </sensor>
+</gazebo>
+<!-- Gazebo sensor plugin for Front LiDAR -->
+<gazebo reference="front_lidar_link">
+  <sensor name="front_lidar" type="gpu_lidar">
+    <pose>0 0 0 0 0 0</pose>
+    <update_rate>10</update_rate>
+    <ray>
+      <scan>
+        <horizontal>
+          <samples>360</samples>
+          <resolution>1.0</resolution>
+          <min_angle>-3.14</min_angle>
+          <max_angle>3.14</max_angle>
+        </horizontal>
+      </scan>
+      <range>
+        <min>0.1</min>
+        <max>30.0</max>
+      </range>
+    </ray>
+  </sensor>
+</gazebo>
+<!-- Gazebo sensor plugin for Rear LiDAR -->
+<gazebo reference="rear_lidar_link">
+  <sensor name="rear_lidar" type="gpu_lidar">
     <pose>0 0 0 0 0 0</pose>
     <update_rate>10</update_rate>
